Commit message: Removed LSM from default.launch; added macbot_sensors to metapackage

File: macbot_description/urdf/robot_textured.xacro (robot description, xacro)
@@ -142,5 +142,5 @@
     </link>
     <!-- LIDAR -->
-    <link name = "ydlidar">
+    <link name = "laser">
         <inertial>
             <mass value = "1" />
@@ -203,5 +203,5 @@
         <origin xyz = "0.0587 0 0.196" rpy = "0 0 0"/>
         <axis xyz = "0 1 0" />
-        <child link = "ydlidar"/>
+        <child link = "laser"/>
         <parent link = "base_link"/>
     </joint>
